Commit message: go2_modified

File: urdf/articulate-trunk-quadruped.urdf (robot description, URDF)
Before this commit: robot articulate-trunk-quadruped, 18 links, 17 joints
Links:
- link base_link: mass 3.456 -> 0.9216
- link base_link_2: mass 3.456 -> 0.9216
- link hip_link: mass 0.603186 -> 1.69646
- link hip_link_2: mass 0.603186 -> 1.69646
- link hip_link_mirrored: mass 0.603186 -> 1.69646
- link hip_link_mirrored_2: mass 0.603186 -> 1.69646
